Commit message: Let the fingers reach the part instead of stopping above it
Desired TCP sits 48 mm above a part centre and the part is 60 mm tall, so
the grasp centre is already 18 mm clear of the top face; fingers that ended
14 mm past the grasp centre stopped 4 mm above the part and never came down
its sides. On arrival the tool read as hovering, and the few millimetres of
residual TCP error had nothing to sit against.

The fingers now run 19 to 63 mm along tool0 z, so they straddle the part
instead. This is appearance only: the fingers carry no collision body, and
tool0_to_tcp stays 35 mm, the same number the project's tool_profile.yaml
declares -- no arrival measurement, structural test or recorded run depends
on how far they extend.

Co-Authored-By: Claude Opus 5 <noreply@anthropic.com>

File: harness/gazebo/scene/ur5e_pick_tool.urdf.xacro (robot description, xacro)
@@ -26,5 +26,10 @@
        declares.  A 6 mm tool plate gap keeps the palm off the wrist_3 mesh,
        which MoveIt would otherwise report as a permanent self-collision.
-       The compact palm and fingers finish at the 35 mm grasp centre. -->
+       Palm spans 0 to 28 mm along tool0 z, fingers 19 to 63 mm, and the grasp
+       centre stays at 35 mm.  The fingers reach past the grasp centre so that
+       on arrival they straddle the sides of a part rather than stopping above
+       it - appearance only.  tool0_to_tcp is unchanged and still the number in
+       the project's tool_profile.yaml; no arrival measurement depends on how
+       far the fingers extend. -->
   <joint name="pick_tool_joint" type="fixed">
     <origin xyz="0 0 0" rpy="0 0 0.0199997"/>
@@ -48,11 +53,11 @@
     </visual>
     <visual name="finger_left">
-      <origin xyz="0 0.034 0.034"/>
-      <geometry><box size="0.016 0.012 0.030"/></geometry>
+      <origin xyz="0 0.034 0.041"/>
+      <geometry><box size="0.016 0.012 0.044"/></geometry>
       <material name="pick_tool_finger"/>
     </visual>
     <visual name="finger_right">
-      <origin xyz="0 -0.034 0.034"/>
-      <geometry><box size="0.016 0.012 0.030"/></geometry>
+      <origin xyz="0 -0.034 0.041"/>
+      <geometry><box size="0.016 0.012 0.044"/></geometry>
       <material name="pick_tool_finger"/>
     </visual>
